File: pcb/bme.kicad_pcb (KiCad board)
At the start: 2 copper layers, 15.2 x 24.8 mm, 22 parts, among them IC1 LSM6DSV320XTR, J1 USB_B_Micro, U1 TP4057

Commit message: Add logo
Parts:
- added G***: LOGO, LOGO, B.Cu at (140.5, 111.0)
